File: MCU-Datalogger/MCU-Datalogger.kicad_sch (KiCad schematic)
At the start: 25 parts, among them U1 24LC1025, U2 24LC1025, U3 DS1337S+, U4 ATMEGA328P-AU, Y1 32.768 KHz, Y2 16 MHz

Commit message: Wriring the second scheet
Other:
- sheet Connectors ports: added D2, D3, D4, D5, D6, D7, D8, GND, MISO, MOSI, RESET, RX, SCK, SDA, TX, Vcc; removed none
Changed lines of the file:
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@@
   (junction (at 232.41 33.02) (diameter 0) (color 0 0 0 0)
+  )
+  (junction (at 110.49 41.91) (diameter 0) (color 0 0 0 0)
   )
   (junction (at 237.49 81.28) (diameter 0) (color 0 0 0 0)
@@
     (stroke (width 0) (type default))
   )
+  (wire (pts (xy 176.53 107.95) (xy 184.15 107.95))
+    (stroke (width 0) (type default))
+  )
   (wire (pts (xy 222.25 33.02) (xy 232.41 33.02))
     (stroke (width 0) (type default))
@@
     (stroke (width 0) (type default))
   )
+  (wire (pts (xy 110.49 41.91) (xy 114.3 41.91))
+    (stroke (width 0) (type default))
+  )
+  (wire (pts (xy 176.53 105.41) (xy 184.15 105.41))
+    (stroke (width 0) (type default))
+  )
   (wire (pts (xy 140.97 50.8) (xy 140.97 63.5))
     (stroke (width 0) (type default))
@@
     (stroke (width 0) (type default))
   )
-  (wire (pts (xy 102.87 41.91) (xy 114.3 41.91))
+  (wire (pts (xy 102.87 41.91) (xy 110.49 41.91))
     (stroke (width 0) (type default))
   )
@@
     (stroke (width 0) (type default))
   )
+  (wire (pts (xy 176.53 109.22) (xy 176.53 107.95))
+    (stroke (width 0) (type default))
+  )
   (wire (pts (xy 222.25 38.1) (xy 222.25 33.02))
     (stroke (width 0) (type default))
@@
     (stroke (width 0) (type default))
   )
+  (wire (pts (xy 110.49 39.37) (xy 110.49 41.91))
+    (stroke (width 0) (type default))
+  )
   (wire (pts (xy 265.43 85.09) (xy 265.43 48.26))
     (stroke (width 0) (type default))
@@
     (effects (font (size 1.27 1.27)) (justify right bottom))
   )
+  (label "D8" (at 207.01 132.08 0) (fields_autoplaced)
+    (effects (font (size 1.27 1.27)) (justify left bottom))
+  )
   (label "D8" (at 185.42 40.64 180) (fields_autoplaced)
     (effects (font (size 1.27 1.27)) (justify right bottom))
@@
     (effects (font (size 1.27 1.27)) (justify right bottom))
   )
+  (label "D6" (at 207.01 127 0) (fields_autoplaced)
+    (effects (font (size 1.27 1.27)) (justify left bottom))
+  )
   (label "SCK" (at 46.99 52.07 180) (fields_autoplaced)
     (effects (font (size 1.27 1.27)) (justify right bottom))
   )
+  (label "MISO" (at 184.15 138.43 180) (fields_autoplaced)
+    (effects (font (size 1.27 1.27)) (justify right bottom))
+  )
   (label "D2" (at 215.9 45.72 0) (fields_autoplaced)
     (effects (font (size 1.27 1.27)) (justify left bottom))
@@
     (effects (font (size 1.27 1.27)) (justify right bottom))
   )
+  (label "RX" (at 184.15 129.54 180) (fields_autoplaced)
+    (effects (font (size 1.27 1.27)) (justify right bottom))
+  )
   (label "Vcc" (at 41.91 154.94 180) (fields_autoplaced)
     (effects (font (size 1.27 1.27)) (justify right bottom))
@@
     (effects (font (size 1.27 1.27)) (justify left bottom))
   )
+  (label "RESET" (at 184.15 140.97 180) (fields_autoplaced)
+    (effects (font (size 1.27 1.27)) (justify right bottom))
+  )
   (label "Vcc" (at 41.91 152.4 180) (fields_autoplaced)
     (effects (font (size 1.27 1.27)) (justify right bottom))
@@
     (effects (font (size 1.27 1.27)) (justify right bottom))
   )
+  (label "MOSI" (at 184.15 135.89 180) (fields_autoplaced)
+    (effects (font (size 1.27 1.27)) (justify right bottom))
+  )
+  (label "D4" (at 207.01 121.92 0) (fields_autoplaced)
+    (effects (font (size 1.27 1.27)) (justify left bottom))
+  )
+  (label "D5" (at 207.01 124.46 0) (fields_autoplaced)
+    (effects (font (size 1.27 1.27)) (justify left bottom))
+  )
   (label "Vcc" (at 76.2 154.94 180) (fields_autoplaced)
     (effects (font (size 1.27 1.27)) (justify right bottom))
   )
+  (label "D2" (at 207.01 116.84 0) (fields_autoplaced)
+    (effects (font (size 1.27 1.27)) (justify left bottom))
+  )
+  (label "D7" (at 207.01 129.54 0) (fields_autoplaced)
+    (effects (font (size 1.27 1.27)) (justify left bottom))
+  )
+  (label "TX" (at 184.15 127 180) (fields_autoplaced)
+    (effects (font (size 1.27 1.27)) (justify right bottom))
+  )
+  (label "SCK" (at 184.15 119.38 180) (fields_autoplaced)
+    (effects (font (size 1.27 1.27)) (justify right bottom))
+  )
   (label "Vcc" (at 170.18 78.74 180) (fields_autoplaced)
     (effects (font (size 1.27 1.27)) (justify right bottom))
   )
+  (label "SDA" (at 184.15 116.84 180) (fields_autoplaced)
+    (effects (font (size 1.27 1.27)) (justify right bottom))
+  )
   (label "D6" (at 215.9 55.88 0) (fields_autoplaced)
     (effects (font (size 1.27 1.27)) (justify left bottom))
@@
     (effects (font (size 1.27 1.27)) (justify left bottom))
   )
+  (label "Vcc" (at 176.53 105.41 180) (fields_autoplaced)
+    (effects (font (size 1.27 1.27)) (justify right bottom))
+  )
   (label "SDA" (at 96.52 149.86 0) (fields_autoplaced)
+    (effects (font (size 1.27 1.27)) (justify left bottom))
+  )
+  (label "D3" (at 207.01 119.38 0) (fields_autoplaced)
     (effects (font (size 1.27 1.27)) (justify left bottom))
   )
@@
     )
   )
+  (symbol (lib_id "power:GND") (at 176.53 109.22 0) (unit 1)
+    (in_bom yes) (on_board yes) (dnp no) (fields_autoplaced)
+    (property "Reference" "#PWR010" (at 176.53 115.57 0)
+      (effects (font (size 1.27 1.27)) hide)
+    )
+    (property "Value" "GND" (at 176.53 114.3 0)
+      (effects (font (size 1.27 1.27)))
+    )
+    (property "Footprint" "" (at 176.53 109.22 0)
+      (effects (font (size 1.27 1.27)) hide)
+    )
+    (property "Datasheet" "" (at 176.53 109.22 0)
+      (effects (font (size 1.27 1.27)) hide)
+    )
+    (pin "1")
+    (instances
+      (project "MCU-Datalogger"
+        (path "/ff08e7c5-b4dc-4c9c-b680-b2226ed71bf7"
+          (reference "#PWR010") (unit 1)
+        )
+      )
+    )
+  )
+  (symbol (lib_id "power:PWR_FLAG") (at 110.49 39.37 0) (unit 1)
+    (in_bom yes) (on_board yes) (dnp no) (fields_autoplaced)
+    (property "Reference" "#FLG03" (at 110.49 37.465 0)
+      (effects (font (size 1.27 1.27)) hide)
+    )
+    (property "Value" "PWR_FLAG" (at 110.49 34.29 0)
+      (effects (font (size 1.27 1.27)))
+    )
+    (property "Footprint" "" (at 110.49 39.37 0)
+      (effects (font (size 1.27 1.27)) hide)
+    )
+    (property "Datasheet" "~" (at 110.49 39.37 0)
+      (effects (font (size 1.27 1.27)) hide)
+    )
+    (pin "1")
+    (instances
+      (project "MCU-Datalogger"
+        (path "/ff08e7c5-b4dc-4c9c-b680-b2226ed71bf7"
+          (reference "#FLG03") (unit 1)
+        )
+      )
+    )
+  )
   (symbol (lib_id "power:GND") (at 85.09 73.66 0) (unit 1)
     (in_bom yes) (on_board yes) (dnp no) (fields_autoplaced)
@@
     )
   )
-  (sheet (at 185.42 119.38) (size 25.4 33.02) (fields_autoplaced)
+  (sheet (at 184.15 101.6) (size 22.86 43.18) (fields_autoplaced)
     (stroke (width 0.1524) (type solid))
     (fill (color 0 0 0 0.0000))
-    (property "Sheetname" "Connectors" (at 185.42 118.6684 0)
+    (property "Sheetname" "Connectors" (at 184.15 100.8884 0)
       (effects (font (size 1.27 1.27)) (justify left bottom))
     )
-    (property "Sheetfile" "Connectors.kicad_sch" (at 185.42 152.9846 0)
+    (property "Sheetfile" "Connectors.kicad_sch" (at 184.15 145.3646 0)
       (effects (font (size 1.27 1.27)) (justify left top))
     )
-    (instances
+    (pin "Vcc" passive (at 184.15 105.41 180)
+      (effects (font (size 1.27 1.27)) (justify left))
+    )
+    (pin "SDA" bidirectional (at 184.15 116.84 180)
+      (effects (font (size 1.27 1.27)) (justify left))
+    )
+    (pin "SCK" passive (at 184.15 119.38 180)
+      (effects (font (size 1.27 1.27)) (justify left))
+    )
+    (pin "GND" passive (at 184.15 107.95 180)
+      (effects (font (size 1.27 1.27)) (justify left))
+    )
+    (pin "D4" bidirectional (at 207.01 121.92 0)
+      (effects (font (size 1.27 1.27)) (justify right))
+    )
+    (pin "D5" bidirectional (at 207.01 124.46 0)
+      (effects (font (size 1.27 1.27)) (justify right))
+    )
+    (pin "D8" bidirectional (at 207.01 132.08 0)
+      (effects (font (size 1.27 1.27)) (justify right))
+    )
+    (pin "D3" bidirectional (at 207.01 119.38 0)
+      (effects (font (size 1.27 1.27)) (justify right))
+    )
+    (pin "D2" bidirectional (at 207.01 116.84 0)
+      (effects (font (size 1.27 1.27)) (justify right))
+    )
+    (pin "D7" bidirectional (at 207.01 129.54 0)
+      (effects (font (size 1.27 1.27)) (justify right))
+    )
+    (pin "TX" output (at 184.15 127 180)
+      (effects (font (size 1.27 1.27)) (justify left))
+    )
+    (pin "RX" input (at 184.15 129.54 180)
+      (effects (font (size 1.27 1.27)) (justify left))
+    )
+    (pin "D6" bidirectional (at 207.01 127 0)
+      (effects (font (size 1.27 1.27)) (justify right))
+    )
+    (pin "RESET" passive (at 184.15 140.97 180)
+      (effects (font (size 1.27 1.27)) (justify left))
+    )
+    (pin "MISO" input (at 184.15 138.43 180)
+      (effects (font (size 1.27 1.27)) (justify left))
+    )
+    (pin "MOSI" input (at 184.15 135.89 180)
+      (effects (font (size 1.27 1.27)) (justify left))
+    )
+    (instances
