File: MCU-Datalogger/MCU-Datalogger.kicad_pcb (KiCad board)
At the start: 2 copper layers, 0 parts

Commit message: Setup pcbnew
Parts:
- added BT1: Battery, Connector_PinHeader_2.54mm:PinHeader_1x02_P2.54mm_Vertical, F.Cu at (252.6, 99.4)
- added C1: 0.1uF, Capacitor_SMD:C_0805_2012Metric, F.Cu at (248.1, 98.5)
- added C2: 22pF, Capacitor_SMD:C_0805_2012Metric, F.Cu at (248.1, 101.6)
- added C3: 22pF, Capacitor_SMD:C_0805_2012Metric, F.Cu at (248.1, 104.6)
- added C4: 0.1uF, Capacitor_SMD:C_0805_2012Metric, F.Cu at (248.1, 107.6)
- added C5: 100nF, Capacitor_SMD:C_0805_2012Metric, F.Cu at (248.1, 110.6)
- added D1: LED, LED_SMD:LED_0805_2012Metric, F.Cu at (252.6, 105.8)
- added D2: LED, LED_SMD:LED_0805_2012Metric, F.Cu at (252.6, 108.8)
- added H1: MountingHole, MountingHole:MountingHole_2.1mm, F.Cu at (228.2, 87.9)
- added H2: MountingHole, MountingHole:MountingHole_2.1mm, F.Cu at (228.2, 93.6)
- added H3: MountingHole, MountingHole:MountingHole_2.1mm, F.Cu at (228.2, 99.4)
- added H4: MountingHole, MountingHole:MountingHole_2.1mm, F.Cu at (228.2, 105.1)
- added J1: Conn_01x04_Pin, Connector_PinHeader_2.54mm:PinHeader_1x04_P2.54mm_Vertical, F.Cu at (264.2, 87.3)
- added J2: Conn_01x04_Pin, Connector_PinHeader_2.54mm:PinHeader_1x04_P2.54mm_Vertical, F.Cu at (268.9, 87.3)
- added J3: Conn_01x09_Pin, Connector_PinHeader_2.54mm:PinHeader_1x09_P2.54mm_Vertical, F.Cu at (259.6, 87.3)
- added J4: Conn_02x03_Odd_Even, Connector_PinHeader_2.54mm:PinHeader_2x03_P2.54mm_Vertical, F.Cu at (264.2, 99.6)
- added R1: 10K, Resistor_SMD:R_0805_2012Metric, F.Cu at (233.3, 86.5)
- added R2: 10K, Resistor_SMD:R_0805_2012Metric, F.Cu at (233.3, 89.4)
- added R3: 4.7k, Resistor_SMD:R_0805_2012Metric, F.Cu at (233.3, 92.4)
- added R4: 4.7k, Resistor_SMD:R_0805_2012Metric, F.Cu at (233.3, 95.3)
- added R5: 330, Resistor_SMD:R_0805_2012Metric, F.Cu at (233.3, 98.3)
- added R6: 10K, Resistor_SMD:R_0805_2012Metric, F.Cu at (233.3, 101.2)
- added R7: 330, Resistor_SMD:R_0805_2012Metric, F.Cu at (233.3, 104.2)
- added U1: 24LC1025, Package_SO:SOIC-8_5.23x5.23mm_P1.27mm, F.Cu at (240.7, 100.4)
- added U2: 24LC1025, Package_SO:SOIC-8_5.23x5.23mm_P1.27mm, F.Cu at (240.7, 107.2)
- added U3: DS1337S+, Footprints:SOIC127P600X175-8N, F.Cu at (251.0, 115.4)
- added U4: ATMEGA328P-AU, Footprints:QFP80P900X900X120-32N, F.Cu at (241.5, 91.0)
- added Y1: 32.768 KHz, Crystal:Crystal_SMD_5032-2Pin_5.0x3.2mm_HandSoldering, F.Cu at (240.6, 113.0)
- added Y2: 16 MHz, Crystal:Crystal_SMD_5032-2Pin_5.0x3.2mm_HandSoldering, F.Cu at (240.6, 117.9)
