File: Breadboard Power Supply/Breadboard Power Supply.kicad_sch (KiCad schematic)
At the start: 17 parts, among them J1 Barrel_Jack_Switch, J2 Screw_Terminal_01x02, J3 Screw_Terminal_01x02, J4 Conn_01x03_Pin, J5 Conn_01x02_Pin, J6 Conn_01x03_Pin, J7 Conn_01x02_Pin, U1 LM317_TO-220, U2 LM7805_TO220

Commit message: Update project
Other:
- company: Mounchili Inteligencia -> Minteligencia
