File: STM32RFUSB/STM32RFUSB.kicad_sch (KiCad schematic)
At the start: 38 parts, among them J1 USB_B_Micro, J2 SWD Connector, J3 SMA, U1 STM32L432KBU6, U2 nRF24L01P, U3 USBLC6-2SC6, U4 XC6206P332MR, Y1 16MHz

Commit message: Create a Project
Parts:
- renumbered C4 to C1, C15 to C10, C18 to C11, C6 to C12, C7 to C13, C10 to C14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
